File: fpga.kicad_sch (KiCad schematic)
At the start: 63 parts, among them CON1 SD_Card_DM3BT, P10 CONN_01X01, P11 CONN_01X01, P12 CONN_01X01, P13 CONN_01X01, P14 CONN_01X01, P15 CONN_01X01, P16 CONN_01X01, P3 CONN_02X04, P4 CONN_02X04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

Commit message: fpga usb clkout pin and one more pin is changed
Connections:
- net CLKOUT: now also U30.D13 (IO_L12P_T1_MRCC_15); no longer U30.A15 (IO_L9N_T1_DQS_AD3N_15)
- net RD#: now also U30.A15 (IO_L9N_T1_DQS_AD3N_15); no longer U30.B14 (IO_L8N_T1_AD10N_15)
Changed lines of the file:
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@@
 	)
 	(no_connect
-		(at 123.19 92.71)
+		(at 123.19 57.15)
 	)
 	(no_connect
@@
 	(wire
 		(pts
-			(xy 120.65 57.15) (xy 123.19 57.15)
-		)
-		(stroke
-			(width 0)
-			(type default)
-		)
-	)
-	(wire
-		(pts
 			(xy 71.12 95.25) (xy 68.58 95.25)
 		)
@@
 	(wire
 		(pts
+			(xy 120.65 92.71) (xy 123.19 92.71)
+		)
+		(stroke
+			(width 0)
+			(type default)
+		)
+	)
+	(wire
+		(pts
 			(xy 35.56 83.82) (xy 29.21 83.82)
 		)
@@
 	)
 	(label "CLKOUT"
-		(at 120.65 44.45 180)
+		(at 120.65 92.71 180)
 		(effects
 			(font
@@
 	)
 	(label "RD#"
-		(at 120.65 57.15 180)
+		(at 120.65 44.45 180)
 		(effects
 			(font
