File: fpga.kicad_sch (KiCad schematic)
At the start: 18 parts, among them U30 XC7A35T-1FTG256C, U35 SolderPad_1_Circle, U38 SolderPad_1_Circle, U4 SolderPad_1_Circle, U41 SolderPad_1_Circle, U42 SolderPad_1_Circle, U43 SolderPad_1_Circle, U44 SolderPad_1_Circle

Commit message: 100t changes design is working tested on a real hardware. Main branch is verified
Parts:
- U30: value XC7A35T-1FTG256C -> XC7A100T-1FTG256C
Changed lines of the file:
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@@
 			)
 		)
-		(property "Value" "XC7A35T-1FTG256C"
+		(property "Value" "XC7A100T-1FTG256C"
 			(at 163.83 22.86 0)
 			(effects
@@
 			)
 		)
-		(property "Value" "XC7A35T-1FTG256C"
+		(property "Value" "XC7A100T-1FTG256C"
 			(at 246.38 22.86 0)
 			(effects
@@
 			)
 		)
-		(property "Value" "XC7A35T-1FTG256C"
+		(property "Value" "XC7A100T-1FTG256C"
 			(at 341.63 22.86 0)
 			(effects
@@
 			)
 		)
-		(property "Value" "XC7A35T-1FTG256C"
+		(property "Value" "XC7A100T-1FTG256C"
 			(at 71.12 142.24 0)
 			(effects
@@
 			)
 		)
-		(property "Value" "XC7A35T-1FTG256C"
+		(property "Value" "XC7A100T-1FTG256C"
 			(at 326.39 184.15 0)
 			(effects
@@
 			)
 		)
-		(property "Value" "XC7A35T-1FTG256C"
+		(property "Value" "XC7A100T-1FTG256C"
 			(at 262.89 181.61 0)
 			(effects
@@
 			)
 		)
-		(property "Value" "XC7A35T-1FTG256C"
+		(property "Value" "XC7A100T-1FTG256C"
 			(at 68.58 27.94 0)
 			(effects
