File: adc.kicad_sch (KiCad schematic)
At the start: 38 parts, among them U39 LP5907-3.0, U8 LTC2292

Commit message: final corrections is done. Working!
Parts:
- R91: value 0 -> 4.7k
- R92: value DNP -> 10k
Other:
- note added: "2/3 VDD clock duty stabilizer 2s complement signed output This helped for better waveform"
Changed lines of the file:
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@@
 	(generator_version "9.0")
 	(paper "A4")
+	(text "2/3 VDD clock duty stabilizer \n2s complement signed output\nThis helped for better waveform"
+		(exclude_from_sim no)
+		(at 52.832 130.81 0)
+		(effects
+			(font
+				(size 1.524 1.524)
+			)
+		)
+	)
 	(junction
 		(at 156.21 48.26)
@@
 			)
 		)
-		(property "Value" "0"
+		(property "Value" "4.7k"
 			(at 72.39 119.38 90)
 			(effects
@@
 			)
 		)
-		(property "Value" "DNP"
+		(property "Value" "10k"
 			(at 72.39 129.54 90)
 			(effects

Commit message: I increased the gap between voltage pours and also corrected signals cutting copper pour. Also not connected gnd occured in some layers are corrected with no copper zoens
Connections:
- net 3V6 renamed 3V8
Changed lines of the file:
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@@
 		)
 	)
-	(hierarchical_label "3V6"
+	(hierarchical_label "3V8"
 		(shape input)
 		(at 44.45 34.29 180)

Commit message: clock buffer and txco source is changed. Clock is clipped sin and fanout says cmos square out but it is better anyways. Also traces are 50 ohm as well. Copper pours other minor thinks are changed as well
Parts:
- R21: value 22 -> 33
Other:
- note added: "Important Note: ECS-TXO-3225MV is pure sin. Adc does not like sin i guess. Other ref designed used clipped more square like sin. That is why clock stabilizer is needed."
Changed lines of the file:
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@@
 		)
 	)
+	(text "Important Note: ECS-TXO-3225MV is pure sin. Adc does not like sin i guess.\nOther ref designed used clipped more square like sin. That is why\nclock stabilizer is needed."
+		(exclude_from_sim no)
+		(at 65.532 148.59 0)
+		(effects
+			(font
+				(size 1.524 1.524)
+			)
+		)
+	)
 	(junction
 		(at 156.21 48.26)
@@
 			)
 		)
-		(property "Value" "22"
+		(property "Value" "33"
 			(at 116.84 78.74 90)
 			(effects

Commit message: lt6232 is done with vias and copper pours are checked
Other:
- moved on the sheet: C163, C164, C165, C166, C167, C168, C19, C20, C216, C217, C218, C219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
