File: adc.kicad_sch (KiCad schematic)
At the start: 38 parts, among them U39 LP5907-3.0, U8 LTC2292

Commit message: minor corrections
Connections:
- net ADC2+: now also R97.2; no longer R99.2
- net ADC2-: now also R99.2; no longer R97.2
Changed lines of the file:
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@@
 		)
 	)
-	(hierarchical_label "ADC2-"
+	(hierarchical_label "ADC2+"
 		(shape input)
 		(at 45.72 68.58 180)
@@
 		)
 	)
-	(hierarchical_label "ADC2+"
+	(hierarchical_label "ADC2-"
 		(shape input)
 		(at 45.72 71.12 180)
