File: clock.kicad_sch (KiCad schematic)
At the start: 10 parts, among them U6 PL133-37, Y2 ECS-TXO-32CSMV

Commit message: lt6232 is done with vias and copper pours are checked
Parts:
- Y2: value ECS-TXO-32CSMV -> ECS ECS-TXO-32CSMV-400
Changed lines of the file:
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@@
 			)
 		)
-		(property "Value" "ECS-TXO-32CSMV"
+		(property "Value" "ECS ECS-TXO-32CSMV-400"
 			(at 120.65 103.124 0)
 			(effects
