File: mixer.kicad_sch (KiCad schematic)
At the start: 31 parts, among them U26 5400BL15B050E, U27 5400BL15B050E, U28 5400BL15B050E, U29 ADL5802

Commit message: IMPORTANT FIX: ADL5802 if output is 200ohm so diff pull ups must be 100 not 50. I have corrected that
Parts:
- R51, R52, R53, R54: value 49.9 -> 100
Other:
- note added: "ADL5801 has 50 ohm network suggestion in its datasheet. However ADL5802 specifically states that it needs 200ohm diff Therefore i will use 100ohm pullup and will not use and transformers since the if will be below 10MHz or so."
- note added: "IMPORTANT: BALUN is 50:50 so output is differential 50 ohm. Also ADL5802 expects 50 ohm differential as well. Therefore rf trace width spacing changes at that part!!!"

Commit message: final corrections is done. Working!
Parts:
- R51, R52, R53, R54: value 100 -> 49.9
Changed lines of the file:
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@@
 			)
 		)
-		(property "Value" "100"
+		(property "Value" "49.9"
 			(at 213.36 83.82 90)
 			(effects
@@
 			)
 		)
-		(property "Value" "100"
+		(property "Value" "49.9"
 			(at 213.36 93.98 90)
 			(effects
@@
 			)
 		)
-		(property "Value" "100"
+		(property "Value" "49.9"
 			(at 213.36 124.46 90)
 			(effects
@@
 			)
 		)
-		(property "Value" "100"
+		(property "Value" "49.9"
 			(at 213.36 134.62 90)
 			(effects

Commit message: I increased the gap between voltage pours and also corrected signals cutting copper pour. Also not connected gnd occured in some layers are corrected with no copper zoens
Other:
- note removed: "ADL5801 has 50 ohm network suggestion in its datasheet. However ADL5802 specifically states that it needs 200ohm diff Therefore i will use 100ohm pullup and will not use and transformers since the if will be below 10MHz or so."

Commit message: changes
Parts:
- U26, U27, U28: value 5400BL15B050E -> 5400BL15B0050001E
Changed lines of the file:
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@@
 			)
 		)
-		(property "Value" "5400BL15B050E"
+		(property "Value" "5400BL15B0050001E"
 			(at 69.85 97.79 0)
 			(effects
@@
 			)
 		)
-		(property "Value" "5400BL15B050E"
+		(property "Value" "5400BL15B0050001E"
 			(at 69.85 121.92 0)
 			(effects
@@
 			)
 		)
-		(property "Value" "5400BL15B050E"
+		(property "Value" "5400BL15B0050001E"
 			(at 69.85 147.32 0)
 			(effects

Commit message: final changes
Other:
- moved on the sheet: C107, C108, C109, C110, C111, C112, C113, C114, C115, C116, C117, C118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

Commit message: DNP components are deleted
Parts:
- removed C107: DNP, Footprints:SMD_0805, symbol fmcw3-rescue:C
Changed lines of the file:
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@@
 	)
 	(junction
-		(at 97.79 40.64)
-		(diameter 0)
-		(color 0 0 0 0)
-	)
-	(junction
 		(at 168.91 119.38)
 		(diameter 0)
@@
 	(wire
 		(pts
-			(xy 96.52 40.64) (xy 97.79 40.64)
+			(xy 96.52 40.64) (xy 101.6 40.64)
 		)
 		(stroke
@@
 	(wire
 		(pts
-			(xy 93.98 43.18) (xy 97.79 43.18)
-		)
-		(stroke
-			(width 0)
-			(type default)
-		)
-	)
-	(wire
-		(pts
 			(xy 180.34 93.98) (xy 208.28 93.98)
 		)
@@
 	(wire
 		(pts
-			(xy 97.79 40.64) (xy 101.6 40.64)
-		)
-		(stroke
-			(width 0)
-			(type default)
-		)
-	)
-	(wire
-		(pts
 			(xy 101.6 114.3) (xy 104.14 114.3)
 		)
@@
 	(wire
 		(pts
-			(xy 97.79 43.18) (xy 97.79 40.64)
-		)
-		(stroke
-			(width 0)
-			(type default)
-		)
-	)
-	(wire
-		(pts
 			(xy 204.47 115.57) (xy 204.47 96.52)
 		)
@@
 	(wire
 		(pts
-			(xy 93.98 48.26) (xy 93.98 43.18)
-		)
-		(stroke
-			(width 0)
-			(type default)
-		)
-	)
-	(wire
-		(pts
 			(xy 73.66 111.76) (xy 71.12 111.76)
 		)
@@
 					(unit 1)
 				)
-			)
-		)
-	)
-	(symbol
-		(lib_id "fmcw3-rescue:C")
-		(at 93.98 52.07 180)
-		(unit 1)
-		(exclude_from_sim no)
-		(in_bom yes)
-		(on_board yes)
-		(dnp no)
-		(property "Reference" "C107"
-			(at 93.345 54.61 0)
-			(effects
-				(font
-					(size 1.27 1.27)
-				)
-				(justify left)
-			)
-		)
-		(property "Value" "DNP"
-			(at 93.345 49.53 0)
-			(effects
-				(font
-					(size 1.27 1.27)
-				)
-				(justify left)
-			)
-		)
-		(property "Footprint" "Footprints:SMD_0805"
-			(at 93.0148 48.26 0)
-			(effects
-				(font
-					(size 0.762 0.762)
-				)
-				(hide yes)
-			)
-		)
-		(property "Datasheet" ""
-			(at 93.98 52.07 0)
-			(effects
-				(font
-					(size 1.524 1.524)
-				)
-			)
-		)
-		(property "Description" ""
-			(at 93.98 52.07 0)
-			(effects
-				(font
-					(size 1.27 1.27)
-				)
-			)
-		)
-		(pin "1"
-		)
-		(pin "2"
-		)
-		(instances
-			(project "fmcw3"
-				(path "/25ababa6-1178-4b22-9ad6-058222120a27/00000000-0000-0000-0000-000059434bd2"
-					(reference "C107")
-					(unit 1)
-				)
-			)
-		)
-	)
-	(symbol
-		(lib_id "fmcw3-rescue:GND")
-		(at 93.98 55.88 0)
-		(unit 1)
-		(exclude_from_sim no)
-		(in_bom yes)
-		(on_board yes)
-		(dnp no)
-		(property "Reference" "#PWR0228"
-			(at 93.98 62.23 0)
-			(effects
-				(font
-					(size 1.27 1.27)
-				)
-				(hide yes)
-			)
-		)
-		(property "Value" "GND"
-			(at 93.98 59.69 0)
-			(effects
-				(font
-					(size 1.27 1.27)
-				)
-			)
-		)
-		(property "Footprint" ""
-			(at 93.98 55.88 0)
-			(effects
-				(font
-					(size 1.524 1.524)
-				)
-			)
-		)
-		(property "Datasheet" ""
-			(at 93.98 55.88 0)
-			(effects
-				(font
-					(size 1.524 1.524)
-				)
-			)
-		)
-		(property "Description" ""
-			(at 93.98 55.88 0)
-			(effects
-				(font
-					(size 1.27 1.27)
-				)
-			)
-		)
-		(pin "1"
-		)
-		(instances
-			(project "fmcw3"
-				(path "/25ababa6-1178-4b22-9ad6-058222120a27/00000000-0000-0000-0000-000059434bd2"
-					(reference "#PWR0228")
-					(unit 1)
-				)
