File: mixer.kicad_sch (KiCad schematic)
At the start: 30 parts, among them U26 5400BL15B0050001E, U27 5400BL15B0050001E, U28 5400BL15B0050001E, U29 ADL5802

Commit message: changes
Connections:
- net IF1+: now also R51.1, U29.3 (OP1+); no longer R52.2, U29.4 (OP1-)
- net IF1-: now also R52.2, U29.4 (OP1-); no longer R51.1, U29.3 (OP1+)
Changed lines of the file:
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@@
 		)
 	)
-	(hierarchical_label "IF1+"
+	(hierarchical_label "IF1-"
 		(shape output)
 		(at 236.22 74.93 0)
@@
 		)
 	)
-	(hierarchical_label "IF1-"
+	(hierarchical_label "IF1+"
 		(shape output)
 		(at 236.22 72.39 0)
