File: opamp_amp.kicad_sch (KiCad schematic)
At the start: 47 parts, among them U2 SolderPad_1_Circle, U31 SolderPad_1_Circle, U34 SolderPad_1_Circle, U45 LT6232, U46 SolderPad_1_Circle, U47 SolderPad_1_Circle, U48 SolderPad_1_Circle, U49 SolderPad_1_Circle, U5 SolderPad_1_Circle

Commit message: lt6232 is done with vias and copper pours are checked
Other:
- moved on the sheet: C13, C15, C16, C32, C33, C34, C36, C37, C38, C39, C40, C41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

Commit message: pcb is checked dnp is deleted copper pours are checked
Connections:
- net IF1+: now also L14.1, R55.1; no longer R55.2, U48.1
- net IF1-: now also L15.1, R56.1; no longer R56.2, U49.1
- net IF2+: now also L12.1, R58.1; no longer R58.2, U46.1
- net IF2-: now also L13.1, R57.1; no longer R57.2, U47.1
- new net: R58.2, U46.1
- new net: R56.2, U49.1
- new net: R55.2, U48.1
- new net: R57.2, U47.1
Changed lines of the file:
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@@
-	)
-	(junction
-		(at 73.66 78.74)
-		(diameter 0)
-		(color 0 0 0 0)
 	)
 	(junction
@@
 	)
 	(junction
+		(at 83.82 45.72)
+		(diameter 0)
+		(color 0 0 0 0)
+	)
+	(junction
 		(at 133.35 86.36)
 		(diameter 0)
@@
 	)
 	(junction
-		(at 74.93 128.27)
+		(at 83.82 78.74)
 		(diameter 0)
 		(color 0 0 0 0)
@@
 	)
 	(junction
-		(at 74.93 152.4)
+		(at 85.09 152.4)
 		(diameter 0)
 		(color 0 0 0 0)
@@
 	)
 	(junction
-		(at 73.66 45.72)
+		(at 85.09 128.27)
 		(diameter 0)
 		(color 0 0 0 0)
@@
 	(wire
 		(pts
+			(xy 83.82 45.72) (xy 87.63 45.72)
+		)
+		(stroke
+			(width 0)
+			(type default)
+		)
+	)
+	(wire
+		(pts
 			(xy 154.94 33.02) (xy 154.94 48.26)
 		)
@@
 	(wire
 		(pts
+			(xy 83.82 50.8) (xy 83.82 45.72)
+		)
+		(stroke
+			(width 0)
+			(type default)
+		)
+	)
+	(wire
+		(pts
 			(xy 154.94 76.2) (xy 151.13 76.2)
 		)
@@
 	(wire
 		(pts
+			(xy 85.09 148.59) (xy 85.09 152.4)
+		)
+		(stroke
+			(width 0)
+			(type default)
+		)
+	)
+	(wire
+		(pts
 			(xy 148.59 64.77) (xy 151.13 64.77)
 		)
@@
 	(wire
 		(pts
-			(xy 82.55 78.74) (xy 87.63 78.74)
+			(xy 82.55 78.74) (xy 83.82 78.74)
 		)
 		(stroke
@@
 	(wire
 		(pts
-			(xy 72.39 78.74) (xy 73.66 78.74)
-		)
-		(stroke
-			(width 0)
-			(type default)
-		)
-	)
-	(wire
-		(pts
 			(xy 181.61 66.04) (xy 186.69 66.04)
 		)
@@
 	(wire
 		(pts
+			(xy 83.82 74.93) (xy 83.82 78.74)
+		)
+		(stroke
+			(width 0)
+			(type default)
+		)
+	)
+	(wire
+		(pts
 			(xy 134.62 115.57) (xy 134.62 109.22)
 		)
@@
 	(wire
 		(pts
-			(xy 83.82 152.4) (xy 88.9 152.4)
+			(xy 83.82 152.4) (xy 85.09 152.4)
+		)
+		(stroke
+			(width 0)
+			(type default)
+		)
+	)
+	(wire
+		(pts
+			(xy 85.09 128.27) (xy 88.9 128.27)
 		)
 		(stroke
@@
 	(wire
 		(pts
+			(xy 85.09 133.35) (xy 85.09 128.27)
+		)
+		(stroke
+			(width 0)
+			(type default)
+		)
+	)
+	(wire
+		(pts
 			(xy 104.14 78.74) (xy 113.03 78.74)
 		)
@@
 	(wire
 		(pts
-			(xy 72.39 45.72) (xy 73.66 45.72)
-		)
-		(stroke
-			(width 0)
-			(type default)
-		)
-	)
-	(wire
-		(pts
 			(xy 134.62 152.4) (xy 134.62 160.02)
 		)
@@
 	(wire
 		(pts
+			(xy 81.28 148.59) (xy 85.09 148.59)
+		)
+		(stroke
+			(width 0)
+			(type default)
+		)
+	)
+	(wire
+		(pts
 			(xy 186.69 143.51) (xy 189.23 143.51)
 		)
@@
 	(wire
 		(pts
-			(xy 73.66 128.27) (xy 74.93 128.27)
-		)
-		(stroke
-			(width 0)
-			(type default)
-		)
-	)
-	(wire
-		(pts
 			(xy 134.62 115.57) (xy 140.97 115.57)
 		)
@@
 	(wire
 		(pts
-			(xy 83.82 128.27) (xy 88.9 128.27)
+			(xy 83.82 128.27) (xy 85.09 128.27)
 		)
 		(stroke
@@
 	(wire
 		(pts
+			(xy 83.82 78.74) (xy 87.63 78.74)
+		)
+		(stroke
+			(width 0)
+			(type default)
+		)
+	)
+	(wire
+		(pts
 			(xy 154.94 86.36) (xy 154.94 76.2)
 		)
@@
 	(wire
 		(pts
-			(xy 73.66 152.4) (xy 74.93 152.4)
-		)
-		(stroke
-			(width 0)
-			(type default)
-		)
-	)
-	(wire
-		(pts
 			(xy 121.92 66.04) (xy 123.19 66.04)
 		)
@@
 	(wire
 		(pts
-			(xy 82.55 45.72) (xy 87.63 45.72)
+			(xy 85.09 152.4) (xy 88.9 152.4)
+		)
+		(stroke
+			(width 0)
+			(type default)
+		)
+	)
+	(wire
+		(pts
+			(xy 82.55 45.72) (xy 83.82 45.72)
 		)
 		(stroke
@@
 	(wire
 		(pts
+			(xy 81.28 133.35) (xy 85.09 133.35)
+		)
+		(stroke
+			(width 0)
+			(type default)
+		)
+	)
+	(wire
+		(pts
 			(xy 74.93 128.27) (xy 76.2 128.27)
 		)
@@
 	(wire
 		(pts
+			(xy 81.28 50.8) (xy 83.82 50.8)
+		)
+		(stroke
+			(width 0)
+			(type default)
+		)
+	)
+	(wire
+		(pts
 			(xy 147.32 33.02) (xy 154.94 33.02)
 		)
@@
 		(pts
 			(xy 154.94 26.67) (xy 154.94 33.02)
+		)
+		(stroke
+			(width 0)
+			(type default)
+		)
+	)
+	(wire
+		(pts
+			(xy 81.28 74.93) (xy 83.82 74.93)
 		)
 		(stroke
@@
 	(hierarchical_label "IF1-"
 		(shape input)
-		(at 73.66 152.4 180)
+		(at 81.28 148.59 180)
 		(effects
 			(font
@@
 	(hierarchical_label "IF2-"
 		(shape input)
-		(at 72.39 78.74 180)
+		(at 81.28 74.93 180)
 		(effects
 			(font
@@
 	(hierarchical_label "IF2+"
 		(shape input)
-		(at 72.39 45.72 180)
+		(at 81.28 50.8 180)
 		(effects
 			(font
@@
 	(hierarchical_label "IF1+"
 		(shape input)
-		(at 73.66 128.27 180)
+		(at 81.28 133.35 180)
 		(effects
 			(font
