File: opamp_amp.kicad_sch (KiCad schematic)
At the start: 47 parts, among them U2 SolderPad_1_Circle, U31 SolderPad_1_Circle, U34 SolderPad_1_Circle, U45 LT6232, U46 SolderPad_1_Circle, U47 SolderPad_1_Circle, U48 SolderPad_1_Circle, U49 SolderPad_1_Circle, U5 SolderPad_1_Circle

Commit message: changes
Parts:
- added JP10, JP11, JP12, JP9: SolderJumper_2_Bridged, Footprints:SolderPad_2_Bridge, symbol Jumper:SolderJumper_2_Bridged
Connections:
- net IF1+: now also R56.2, JP12.2 (B); no longer L14.1, R55.1
- net IF1-: now also R55.2, JP11.1 (A); no longer L15.1, R56.1
- net IF2+: now also R57.2, JP9.2 (B); no longer L12.1, R58.1
- net IF2-: now also R58.2, JP10.1 (A); no longer L13.1, R57.1
- net at U46.1: now also JP10.2 (B); no longer R58.2
- net at U49.1: now also JP12.1 (A); no longer R56.2
- net at U48.1: now also JP11.2 (B); no longer R55.2
- net at U47.1: now also JP9.1 (A); no longer R57.2
- new net: L12.1, R58.1
- new net: L14.1, R55.1
- new net: L13.1, R57.1
- new net: L15.1, R56.1
Other:
- moved on the sheet: U46, U47, U48, U49

Commit message: 100t changes design is working tested on a real hardware. Main branch is verified
Parts:
- R26, R28, R31, R38: value 500 -> 1k
Changed lines of the file:
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@@
 			)
 		)
-		(property "Value" "500"
+		(property "Value" "1k"
 			(at 127 78.74 90)
 			(effects
@@
 			)
 		)
-		(property "Value" "500"
+		(property "Value" "1k"
 			(at 128.27 152.4 90)
 			(effects
@@
 			)
 		)
-		(property "Value" "500"
+		(property "Value" "1k"
 			(at 127 45.72 90)
 			(effects
@@
 			)
 		)
-		(property "Value" "500"
+		(property "Value" "1k"
 			(at 128.27 128.27 90)
 			(effects
