File: fmcw3.kicad_sch (KiCad schematic)
At the start: 0 parts

Commit message: minor corrections
Other:
- sheet tx ports: added TX_LO; removed TX_COUPLED
Changed lines of the file:
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@@
 			)
 		)
-		(pin "TX_COUPLED" output
+		(pin "TX_LO" output
 			(at 203.2 38.1 0)
 			(effects
