File: tx.kicad_sch (KiCad schematic)
At the start: 53 parts, among them U1 ADF4158, U10 HMC431LP4, U12 PAT1220-3dB, U14 TQP5525, U15 SMA, U3 PAT1220-6dB, U36 SolderPad_1_Circle, U7 TLV172DCK

Commit message: minor corrections
Connections:
- net TX_COUPLED renamed TX_LO
Changed lines of the file:
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@@
 		)
 	)
-	(hierarchical_label "TX_COUPLED"
+	(hierarchical_label "TX_LO"
 		(shape output)
 		(at 358.14 156.21 270)
